File: pcb/FDRbox.sch (KiCad schematic (older format))
At the start: 18 parts, among them P1 USB_B, P2 ICSP, U1 PIC16F1455, U2 4051

Commit message: Added note to PCB schematic
Other:
- note added: "Faders are connected according to grey code.\nFDR_6 and FDR_7, FDR_4 and FDR_5 have to be swapped.\nUse regular order in next revision."
- note removed: "Faders are connected according to grey code."
Changed lines of the file:
@@
 LIBS:valves
 LIBS:PIC16F145x
+LIBS:FDRbox-cache
 EELAYER 25 0
 EELAYER END
@@
 	0    -1   -1   0
 $EndComp
-Text Notes 6800 1800 0    60   ~ 0
-Faders are connected according to grey code.
+Text Notes 6900 1800 0    60   ~ 0
+Faders are connected according to grey code.\nFDR_6 and FDR_7, FDR_4 and FDR_5 have to be swapped.\nUse regular order in next revision.
 $EndSCHEMATC
